File: reaktor51_led/reaktor51_led.kicad_pcb (KiCad board)
At the start: 2 copper layers, 57 x 65 mm, 5 parts, among them SW1 SW_SPST

Commit message: reaktor51_led rev1 rc2
Parts:
- BT1: value Battery_Cell -> CR2032
- SW1: value SW_SPST -> Pushbutton
Changed lines of the file:
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@@
 	)
 	(paper "A4")
+	(title_block
+		(title "Reaktor51 LED")
+		(date "2024-04-26")
+		(rev "1")
+		(comment 1 "Aurhor: Inge Aune Paulsen")
+	)
 	(layers
 		(0 "F.Cu" signal)
@@
 	(net 1 "Net-(BT1-+)")
 	(net 2 "GND")
-	(net 3 "Net-(SW1-B)")
+	(net 3 "Net-(R1-Pad2)")
 	(net 4 "Net-(D1-A)")
 	(footprint "Button_Switch_THT:SW_PUSH_6mm"
 		(layer "F.Cu")
 		(at 174 71.75 90)
-		(descr "https://www.omron.com/ecb/products/pdf/en-b3f.pdf")
+		(descr "Generic 6mm SW tactile push button")
 		(tags "tact sw push 6mm")
 		(property "Reference" "SW1"
@@
 			)
 		)
-		(property "Value" "SW_SPST"
+		(property "Value" "Pushbutton"
 			(at 3.75 6.7 -90)
 			(layer "F.Fab")
@@
 			)
 		)
-		(property "Description" "Single Pole Single Throw (SPST) switch"
+		(property "Description" "Push button switch, generic, two pins"
 			(at 0 0 90)
 			(unlocked yes)
@@
 			)
 		)
-		(sheetname "Root")
-		(sheetfile "reaktor51_led.kicad_sch")
 		(attr through_hole)
 		(fp_line
@@
 			(remove_unused_layers no)
 			(net 1 "Net-(BT1-+)")
-			(pinfunction "A")
+			(pinfunction "1")
 			(pintype "passive")
 		)
@@
 			(remove_unused_layers no)
 			(net 1 "Net-(BT1-+)")
-			(pinfunction "A")
+			(pinfunction "1")
 			(pintype "passive")
 		)
@@
 			(layers "*.Cu" "*.Mask")
 			(remove_unused_layers no)
-			(net 3 "Net-(SW1-B)")
-			(pinfunction "B")
+			(net 3 "Net-(R1-Pad2)")
+			(pinfunction "2")
 			(pintype "passive")
 		)
@@
 			(layers "*.Cu" "*.Mask")
 			(remove_unused_layers no)
-			(net 3 "Net-(SW1-B)")
-			(pinfunction "B")
+			(net 3 "Net-(R1-Pad2)")
+			(pinfunction "2")
 			(pintype "passive")
 		)
-		(model "${KICAD6_3DMODEL_DIR}/Button_Switch_THT.3dshapes/SW_PUSH_6mm.wrl"
+		(model "${KICAD8_3DMODEL_DIR}/Button_Switch_THT.3dshapes/SW_PUSH_6mm.wrl"
 			(offset
 				(xyz 0 0 0)
@@
 			)
 		)
-		(property "Value" "Battery_Cell"
+		(property "Value" "CR2032"
 			(at 15 13 90)
 			(layer "F.Fab")
@@
 			)
 		)
-		(property "Description" ""
+		(property "Description" "Single-cell battery"
 			(at 0 0 -90)
 			(unlocked yes)
@@
 			)
 		)
-		(sheetname "Root")
-		(sheetfile "reaktor51_led.kicad_sch")
 		(attr through_hole)
 		(fp_line
@@
 		(fp_arc
 			(start 3.5 3.25)
-			(mid 3.80926 3.345922)
+			(mid 3.809279 3.345913)
 			(end 4.01 3.6)
 			(stroke
@@
 			(pintype "passive")
 		)
-		(model "${KICAD6_3DMODEL_DIR}/Battery.3dshapes/BatteryHolder_Keystone_103_1x20mm.wrl"
+		(model "${KICAD8_3DMODEL_DIR}/Battery.3dshapes/BatteryHolder_Keystone_103_1x20mm.wrl"
 			(offset
 				(xyz 0 0 0)
@@
 			)
 		)
-		(property "Description" ""
+		(property "Description" "Resistor"
 			(at 0 0 0)
 			(unlocked yes)
@@
 			)
 		)
-		(property ki_fp_filters "R_*")
-		(sheetname "Root")
-		(sheetfile "reaktor51_led.kicad_sch")
 		(attr through_hole)
 		(fp_line
@@
 			(layers "*.Cu" "*.Mask")
 			(remove_unused_layers no)
-			(net 3 "Net-(SW1-B)")
+			(net 3 "Net-(R1-Pad2)")
 			(pintype "passive")
 		)
-		(model "${KICAD6_3DMODEL_DIR}/Resistor_THT.3dshapes/R_Axial_DIN0207_L6.3mm_D2.5mm_P10.16mm_Horizontal.wrl"
+		(model "${KICAD8_3DMODEL_DIR}/Resistor_THT.3dshapes/R_Axial_DIN0207_L6.3mm_D2.5mm_P10.16mm_Horizontal.wrl"
 			(offset
 				(xyz 0 0 0)
@@
 			)
 		)
-		(property "Description" ""
+		(property "Description" "Light emitting diode"
 			(at 0 0 -90)
 			(unlocked yes)
@@
 			)
 		)
-		(property ki_fp_filters "LED* LED_SMD:* LED_THT:*")
-		(sheetname "Root")
-		(sheetfile "reaktor51_led.kicad_sch")
 		(attr through_hole)
 		(fp_line
@@
 			(pintype "passive")
 		)
-		(model "${KICAD6_3DMODEL_DIR}/LED_THT.3dshapes/LED_D5.0mm.wrl"
+		(model "${KICAD8_3DMODEL_DIR}/LED_THT.3dshapes/LED_D5.0mm.wrl"
 			(offset
 				(xyz 0 0 0)
