File: reaktor51_game/reaktor51_game.kicad_pcb (KiCad board)
At the start: 2 copper layers, 54 x 65 mm, 17 parts, among them SW1 SW_Push_LED, SW2 SW_Push_LED, SW3 SW_Push_LED, SW4 SW_Push_LED, U1 ATtiny13A-P

Commit message: Reaktor51 Memory Game REV2
Parts:
- C1, C2: value C -> 1u
- R5: value 1k -> 4k7
Other:
- board text added: "1"
- board text added: "2"
- board text added: "3"
- board text added: "4"
- board text added: "IngeP 2025"
- board text added: "MEMORY GAME"
- board text added: "REV2"
- board text removed: "IngeP 2024"
- board text removed: "REACTION GAME"
- board text removed: "REV1"
