File: reaktor51_game/reaktor51_game.kicad_sch (KiCad schematic)
At the start: 15 parts, among them SW1 SW_Push_LED, SW2 SW_Push_LED, SW3 SW_Push_LED, SW4 SW_Push_LED, U1 ATtiny13A-P

Commit message: Reaktor51 Memory Game REV2
Parts:
- BT1: Digikey 36-103-ND -> (none); Link (none) -> https://www.digikey.no/en/products/detail/keystone-electron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
- C1, C2: Link (none) -> https://www.digikey.no/en/products/detail/tdk-corporation/F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; MnfPnr (none) -> FG18X7R1E105KRT00; Mnfr (none) -> TDK
- LS1: Link (none) -> https://www.aliexpress.com/item/1005004932492920.html; MnfPnr (none) -> 1407 Piezoelectric Passive Buzzer 14x4mm 7.5mm; Mnfr (none) -> AliExpress
- R1, R2, R3, R4, R6: Digikey CF14JT150RCT-ND -> (none); Link (none) -> https://www.digikey.no/en/products/detail/stackpole-electro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
- R5: value 1k -> 4k7; Digikey CF14JT150RCT-ND -> (none); Link (none) -> https://www.digikey.no/en/products/detail/stackpole-electro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; MnfPnr CF14JT150R -> CF14JT4K70
- SW1, SW2, SW3, SW4: Link (none) -> https://www.aliexpress.com/item/1005003507477622.html; MnfPnr (none) -> 12*12*7.3mm RED; Mnfr (none) -> AliExpress
- U1: Link (none) -> https://www.digikey.no/en/products/detail/microchip-technol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; MnfPnr (none) -> ATtiny13A-PU; Mnfr (none) -> Microchip Technology
Other:
- title: Reaktor51 Game -> Reaktor51 Memory Game
